File: boards/unoQ/layout/unoQ/layout.kicad_pcb (KiCad board)
At the start: 2 copper layers, 68.6 x 53.3 mm, 428 parts, among them IC1 ?, IC2 ?, IC3 ?, IC4 ?, IC5 ?, IC6 ?, IC7 ?, J1 ?, J2 ?, J3 , J4 , Q1 ?, Q2 ?, Q3 ?, Q4 ?, Q5 ?, U1 ?, U2 ?, Y1 16MHz, Y2 32kHz

Commit message: fix CI
Parts:
- D1, D2, D3: value ? -> SX34
- D10, D11, D12, D13, D14, D15, D16, D17, D18, D19, D20, D21, D22, D23, D24, D25, D26, D27, D28, D29, D30, D31, D32, D33, D34, D35, D36, D37, D38, D39, D40, D41, D42, D43, D44, D5, D6, D7, D8, D9: value ? -> DF2B7ASL
- D4: value ? -> RCLAMP0522P.TCT
- D45: value ? -> PJGBLC24C
- D46, D47, D48, D49, D50, D51, D52, D53, D54: value ? -> RCLAMP0524PATCT
- D55, D56, D57, D58: value ? -> PESD5V0X1BL,315
- IC1: value ? -> LMR51440SDRRR
- IC2, IC3: value ? -> TPS62A02APDDCR
- IC4: value ? -> RCLAMP3654PATCT
- IC5: value ? -> MT53E512M32D1ZW-046 AUT:B
- IC6: value ? -> 74LVC1G3157DW-7
- IC7: value ? -> STM32U585AII6TR
- J1, J2: value ? -> CLE-130-01-G-DV-P-TR
- L1, L2: value ? -> TFM252012ALMA1R0MTAA
- L3: value ? -> NRS8030T3R3MJGJ
- Q1: value ? -> SMMBT3904WT1G
Other:
- copper layers 2 -> 4
